File: Hardware/FOC_Power.kicad_sch (KiCad schematic)
At the start: 10 parts, among them U1 STM32F405RGTx

Commit message: Init Files
Parts:
- C? (x2): value (none) -> 2.2uF
- C?: value (none) -> 0.1uF
- Y?: value (none) -> CSTCE12M0G15L08-R0; footprint (none) -> Crystal:OSC_CSTCE12M0G15L08-R0
Connections:
- net GND: now also Y?.2
- net PH0: now reaches Y?.1
- net PH0: now also U1.5 (PH0)
- net PH1: now reaches Y?.3
- net PH1: now also U1.6 (PH1)
- net BOOT0: now reaches U1.60 (BOOT0)
- net NRST: now reaches U1.7 (NRST)
Other:
- moved on the sheet: C?, Y?

Commit message: Init FreeRTOS
Parts:
- added C18, C27, C29, C30, C33: 10uF, Capacitor_SMD:C_0402_1005Metric, symbol Device:C
- added C19, C21: 4.7uF, Capacitor_SMD:C_0402_1005Metric, symbol Device:C
- added C20, C22, C23, C24, C25, C28, C31, C7, C8, C9: 0.1uF, Capacitor_SMD:C_0402_1005Metric, symbol Device:C
- added C26: 100pF, Capacitor_SMD:C_0402_1005Metric, symbol Device:C
- added C32: 10nF, Capacitor_SMD:C_0402_1005Metric, symbol Device:C
- added D2: LED, LED_SMD:LED_0402_1005Metric, symbol Device:LED
- added D3, D4, D7: B5819WS, Diode_SMD:D_SOD-323, symbol Device:D
- added H1, H2, H3, H4: Hole, Userlib:Hole, symbol UserLIB:Hole
- added J2: USB_C_Receptacle_USB2.0, Connector_USB:USB_C_Receptacle_Palconn_UTC16-G, symbol Connector:USB_C_Receptacle_USB2.0
- added J3: XT30, Connector_AMASS:XT30_SMD, symbol Connector:Conn_01x02_Male
- added J7: Conn_01x05_Male, Connector_JST:JST_SUR_SM05B-SURS-TF_1x05-1MP_P0.80mm_Horizontal, symbol Connector:Conn_01x05_Male
- added J8: Conn_01x02_Male, Connector_JST:JST_SUR_SM02B-SURS-TF_1x02-1MP_P0.80mm_Horizontal, symbol Connector:Conn_01x02_Male
- added J9: Conn_01x04_Male, Connector_JST:JST_SUR_SM04B-SURS-TF_1x04-1MP_P0.80mm_Horizontal, symbol Connector:Conn_01x04_Male
- added JP1: SolderJumper_3_Open, Jumper:SolderJumper-3_P1.3mm_Open_RoundedPad1.0x1.5mm, symbol Jumper:SolderJumper_3_Open
- added L1: 6.8uH, Inductor_SMD:L_0805_2012Metric, symbol Device:L
- added R10, R18, R4, R8, R9: 4.7K, Resistor_SMD:R_0402_1005Metric, symbol Device:R
- added R11, R12, R13, R15, R19, R3: 10K, Resistor_SMD:R_0402_1005Metric, symbol Device:R
- added R14: 1M, Resistor_SMD:R_0402_1005Metric, symbol Device:R
- added R16: 1.8K, Resistor_SMD:R_0402_1005Metric, symbol Device:R
- added R17: 560K, Resistor_SMD:R_0402_1005Metric, symbol Device:R
- added R20, R21: 5K1, Resistor_SMD:R_0402_1005Metric, symbol Device:R
- added S1: RST, Button_Switch_SMD:SKRK, symbol UserLIB:SKRKAEE010_Button
- added S2: ENT, Button_Switch_SMD:SKRK, symbol UserLIB:SKRKAEE010_Button
- added S3: SEL, Button_Switch_SMD:SKRK, symbol UserLIB:SKRKAEE010_Button
- added U3: ME3116, Package_TO_SOT_SMD:SOT-23-6, symbol UserLIB:ME3116
- added U4: CP2102N-Axx-xQFN20, Package_DFN_QFN:SiliconLabs_QFN-20-1EP_3x3mm_P0.5mm_EP1.8x1.8mm, symbol Interface_USB:CP2102N-Axx-xQFN20
- added U5: OLED-12880, Userlib:OLED-12880, symbol UserLIB:OLED-12880
- added U6: LP2992-3V3, Package_TO_SOT_SMD:SOT-23-5, symbol UserLIB:LP2992-3V3
- C10, C11, C12, C13, C14, C15, C16, C17: renamed from C?; footprint (none) -> Capacitor_SMD:C_0402_1005Metric
- gave numbers to parts that had none: 1
Connections:
- net +3V3: now also C21.1, C22.1, C31.1, C33.1, J7.1 (Pin_1), J9.1 (Pin_1), JP1.1 (A), R10.2, R11.2, R12.1, R13.1, R18.2, R19.1, R3.1, R4.2, R8.2, R9.2, U4.6 (VDD), U4.9 (~{RST}), U5.4 (VDD), U6.5 (OUT)
- net BOOT0: now also JP1.2 (C)
- net GND: now also C18.2, C19.2, C20.2, C21.2, C22.2, C25.1, C27.1, C28.1, C29.2, C30.2, C31.2, C32.1, C33.2, C7.2, C8.2, C9.2, D4.2 (A), H1.1, H2.1, H3.1, H4.1, J2.A1 (GND), J2.A12 (GND), J2.B1 (GND), J2.B12 (GND), J2.S1 (SHIELD), J3.1 (Pin_1), J7.5 (Pin_5), J9.4 (Pin_4), JP1.3 (B), R16.2, R17.2, R20.2, R21.2, S1.1, S2.1, S3.1, U3.2 (GND), U4.12 (GND), U4.21 (GND), U4.3 (GND), U5.12 (VSS), U5.7 (CS), U5.9 (DC), U6.2 (GND)
- net NRST: now also C7.1, R3.2, S1.2
- net SOA1: now reaches U1.15 (PA1)
- net SOB1: now reaches U1.16 (PA2)
- net SOC1: now reaches U1.17 (PA3)
- net SOA0: now reaches U1.20 (PA4)
- net SOB0: now reaches U1.21 (PA5)
- net SOC0: now reaches U1.22 (PA6)
- net INLA1: now reaches U1.23 (PA7)
- net INLB0: now reaches U1.26 (PB0)
- net INLC0: now reaches U1.27 (PB1)
- net I2C2_SCL: now reaches U1.29 (PB10)
- net I2C2_SCL: now also R8.1
- net KEY_ENT: now reaches U1.3 (PC14)
- net KEY_ENT: now also C8.1, R12.2, S2.2
- net I2C2_SDA: now reaches U1.30 (PB11)
- net I2C2_SDA: now also R4.1
- net INLA0: now reaches U1.34 (PB13)
- net INLB1: now reaches U1.35 (PB14)
- net INLC1: now reaches U1.36 (PB15)
- net INHA1: now reaches U1.37 (PC6)
- net INHB1: now reaches U1.38 (PC7)
- net INHC1: now reaches U1.39 (PC8)
- net KEY_SEL: now reaches U1.4 (PC15)
- net KEY_SEL: now also C9.1, R13.2, S3.2
- net EN0: now reaches U1.40 (PC9)
- net INHC0: now reaches U1.41 (PA8)
- net INHB0: now reaches U1.42 (PA9)
- net INHA0: now reaches U1.43 (PA10)
- net CAN1_RX: now reaches U1.44 (PA11)
- net CAN1_RX: now also J8.2 (Pin_2)
- net CAN1_TX: now reaches U1.45 (PA12)
- net CAN1_TX: now also J8.1 (Pin_1)
- net CAL0: now reaches U1.46 (PA13)
- net USART3_TX: now reaches U1.51 (PC10)
- net USART3_TX: now also J9.3 (Pin_3)
- net USART3_RX: now reaches U1.52 (PC11)
- net USART3_RX: now also J9.2 (Pin_2)
- net User_LED: now reaches U1.53 (PC12)
- net User_LED: now also D2.1 (K)
- net SPI1_SCK: now reaches U1.55 (PB3)
- net SPI1_SCK: now also J7.4 (Pin_4)
- net SPI1_MISO: now reaches U1.56 (PB4)
- net SPI1_MISO: now also J7.3 (Pin_3)
- net SPI1_MOSI: now reaches U1.57 (PB5)
- net SPI1_MOSI: now also J7.2 (Pin_2)
- net USART1_TX: now reaches U1.58 (PB6)
- net USART1_TX: now also U4.17 (RXD)
- net USART1_RX: now reaches U1.59 (PB7)
- net USART1_RX: now also U4.18 (TXD)
- net I2C1_SCL: now reaches U1.61 (PB8)
- net I2C1_SCL: now also R10.1, U5.10 (SCL)
- net I2C1_SDA: now reaches U1.62 (PB9)
- net I2C1_SDA: now also R9.1, U5.11 (SDA)
- net EN1: now reaches U1.8 (PC0)
- net CAL1: now reaches U1.9 (PC1)
- new net: C32.2, U6.4 (BYPASS)
- new net: C26.2, R15.2, R16.1, U3.3 (FB)
- new net: C23.1, C24.1, D4.1 (K), L1.1, U3.6 (SW)
- new net: C29.1, U5.3 (VCCOMH)
- new net: R18.1, U5.5 (IM1)
- new net: R17.1, U5.6 (IREF)
- new net: C30.1, R19.2, U5.8 (RES)
- new net: J2.A5 (CC1), R20.1
- new net: J2.B5 (CC2), R21.1
- new net: C18.1, D3.1 (K), R14.1, U3.5 (VIN)
- new net: R14.2, U3.4 (EN)
- new net: D2.2 (A), R11.1
- new net: C23.2, C24.2, U3.1 (BS)
- new net +12V: D3.2 (A), J3.2 (Pin_2)
- new net +5V: C19.1, C20.1, C25.2, C26.1, C27.2, C28.2, D7.1 (K), L1.2, R15.1, U4.7 (VREGIN), U4.8 (VBUS), U5.2 (VPP), U6.1 (VIN), U6.3 (EN)
- new net D+: J2.A6 (D+), J2.B6 (D+), U4.4 (D+)
- new net D-: J2.A7 (D-), J2.B7 (D-), U4.5 (D-)
- new net VBUS: D7.2 (A), J2.A4 (VBUS), J2.A9 (VBUS), J2.B4 (VBUS), J2.B9 (VBUS)
- no-connect marks 0 -> 13
Other:
- moved on the sheet: C10, C11, C12, C13, C14, C15, C16, C17, Y1
