File: Hardware/Motor1.kicad_sch (KiCad schematic)
At the start: 36 parts, among them J1 Motor0, Q1 IRF7480M, Q2 IRF7480M, Q3 IRF7480M, Q4 IRF7480M, Q5 IRF7480M, Q6 IRF7480M, U2 DRV8323HRTAR

Commit message: Init FreeRTOS
Parts:
- removed R? (x2): 4.7K, Resistor_SMD:R_2512_6332Metric, symbol Device:R
- added C60, C61, C62, C63, C64, C65, C66, C67: 220uF, Capacitor_SMD:C_0805_2012Metric, symbol Device:C
- added R39, R40, R41, R42, R43, R44: 2.2R, Resistor_SMD:R_0402_1005Metric, symbol Device:R
- C34, C35, C36: renamed from C?; footprint (none) -> Capacitor_SMD:C_0402_1005Metric
- C37, C38, C39: renamed from C?; footprint (none) -> Capacitor_SMD:C_0603_1608Metric
- C40, C41, C42, C43: renamed from C?; footprint (none) -> Capacitor_SMD:C_0805_2012Metric
- D1: footprint LED_SMD:LED_0603_1608Metric -> LED_SMD:LED_0402_1005Metric
- J1: footprint Connector_AMASS:AMASS_MR30PW-M_1x03_P3.50mm_Horizontal -> Connector_AMASS:MR30_SMD
- J4: renamed from J?; footprint (none) -> Connector_JST:JST_SUR_SM04B-SURS-TF_1x04-1MP_P0.80mm_Horizontal
- gave numbers to parts that had none: 3
Connections:
- net +12V: now also C60.1, C61.1, C62.1, C63.1, C64.1, C65.1, C66.1, C67.1
- net GHA: now also R39.1; no longer Q1.2 (G)
- net GHB: now also R41.1; no longer Q3.2 (G)
- net GHC: now also R43.1; no longer Q5.2 (G)
- net GLA: now also R40.1; no longer Q2.2 (G)
- net GLB: now also R42.1; no longer Q4.2 (G)
- net GLC: now also R44.1; no longer Q6.2 (G)
- net GND: now also C60.2, C61.2, C62.2, C63.2, C64.2, C65.2, C66.2, C67.2
- new net: Q3.2 (G), R41.2
- new net: Q2.2 (G), R40.2
- new net: Q1.2 (G), R39.2
- new net: Q5.2 (G), R43.2
- new net: Q4.2 (G), R42.2
- new net: Q6.2 (G), R44.2
Other:
- moved on the sheet: J1, J4, Q1, Q2, Q3, Q4, Q5, Q6, R5, R6, R7
